File: hardware/kicad/EyeNode/EyeNode.kicad_pcb (KiCad board)
At the start: 2 copper layers, 110 x 90 mm, 43 parts, among them J1 12V IN logica, J10 RS485 OUT, J11 AUX I2C/A6, J2 5-6V IN servo, J3 SERVO A_LR, J4 SERVO A_UD, J5 SERVO A_LID, J6 SERVO B_LR, J7 SERVO B_UD, J8 SERVO B_LID, J9 RS485 IN, SW1 ADDR, U1 R-78E5.0-0.5, U2 MAX485E

Commit message: changed image and setup
Parts:
- removed C6: 100nF, Capacitor_SMD:C_1206_3216Metric
- removed J10: RS485 OUT, TerminalBlock_Phoenix:TerminalBlock_Phoenix_MKDS-1,5-3-5.08_1x03_P5.08mm_Horizontal
- removed J9: RS485 IN, TerminalBlock_Phoenix:TerminalBlock_Phoenix_MKDS-1,5-3-5.08_1x03_P5.08mm_Horizontal
- removed JP1: TERM 120R, Connector_PinHeader_2.54mm:PinHeader_1x02_P2.54mm_Vertical
- removed R7: 120, Resistor_SMD:R_1206_3216Metric
- removed U2: MAX485E, Package_SO:SOIC-8_3.9x4.9mm_P1.27mm
Connections:
- A1 pad 10: /RS485_TX -> unconnected-(A1-D7-Pad10)
- A1 pad 11: /RS485_RX -> unconnected-(A1-D8-Pad11)
- A1 pad 7: /RS485_DE -> unconnected-(A1-D4-Pad7)
Routing:
- net /+5V: track 150.6 -> 88.3 mm, vias 1 -> 0
- net /RS485_B: track 52.6 -> 0.00 mm
- net /GND: track 366.2 -> 314.1 mm, vias 2 -> 1
- net /RS485_DE: track 49.2 -> 0.00 mm, vias 1 -> 0
- net /RS485_A: track 41.2 -> 0.00 mm
- net /RS485_TX: track 39.5 -> 0.00 mm
- net /RS485_RX: track 34.0 -> 0.00 mm
- net /ADDR1: track 110.4 -> 93.3 mm
- net /VSERVO: track 170.9 -> 160.9 mm
- net /TERM: track 7.02 -> 0.00 mm
- net /VLOGIC: track 17.6 -> 13.5 mm
- net /ADDR2: track 95.6 -> 92.3 mm
- net /PWM_A_UD: track 52.4 -> 54.8 mm
- net /PWM_A_LID: track 43.8 -> 46.1 mm
- net /AUX_SCL: track 73.4 -> 75.6 mm
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Other:
- board text added: "EyeNode v0.2 - Idra di Guerra"
- board text removed: "EyeNode v0.1 - Idra di Guerra"
- board text removed: "IN: A B GND"
- board text removed: "OUT: A B GND"
