File: hardware/kicad/EyeNode/EyeNode.kicad_sch (KiCad schematic)
At the start: 43 parts, among them J1 12V IN logica, J10 RS485 OUT, J11 AUX I2C/A6, J2 5-6V IN servo, J3 SERVO A_LR, J4 SERVO A_UD, J5 SERVO A_LID, J6 SERVO B_LR, J7 SERVO B_UD, J8 SERVO B_LID, J9 RS485 IN, SW1 ADDR, U1 R-78E5.0-0.5, U2 MAX485E

Commit message: changed image and setup
Parts:
- removed C6: 100nF, Capacitor_SMD:C_1206_3216Metric, symbol Device:C
- removed J10: RS485 OUT, TerminalBlock_Phoenix:TerminalBlock_Phoenix_MKDS-1,5-3-5.08_1x03_P5.08mm_Horizontal, symbol Connector_Generic:Conn_01x03
- removed J9: RS485 IN, TerminalBlock_Phoenix:TerminalBlock_Phoenix_MKDS-1,5-3-5.08_1x03_P5.08mm_Horizontal, symbol Connector_Generic:Conn_01x03
- removed JP1: TERM 120R, Connector_PinHeader_2.54mm:PinHeader_1x02_P2.54mm_Vertical, symbol Jumper:Jumper_2_Open
- removed R7: 120, Resistor_SMD:R_1206_3216Metric, symbol Device:R
- removed U2: MAX485E, Package_SO:SOIC-8_3.9x4.9mm_P1.27mm, symbol Interface_UART:MAX485E
Connections:
- net RS485_DE: no longer names the net of A1.7 (D4)
- net RS485_RX: no longer names the net of A1.11 (D8)
- net RS485_TX: no longer names the net of A1.10 (D7)
- no-connect marks 9 -> 12
Other:
- note removed: "BUS RS-485 (sincronizzazione teste)"
